File: HW/ES3ink.kicad_sch (KiCad schematic)
At the start: 72 parts, among them J1 USB_C_Receptacle_USB2.0, J2 Conn_01x24_Pin, J2 USB_C_Receptacle_USB2.0, J3 Conn_01x02_Pin, J4 Conn_01x04_Socket, Q1 DMG3415U-7, Q2 SI1308EDL-T1-GE3, Q3 DMG3415U-7, Q4 SI2305, SW1 RESET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

Commit message: Component update
Parts:
- D1, D2, D3: value MBR0520LT -> MBR0530-TP
- L1: value 68uH -> 10uH/1A; Mouser (none) -> https://eu.mouser.com/ProductDetail/Murata-Electronics/LQH4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
- Q1: value DMG3415U-7 -> AO3401A
- R10: value 10R -> 0R
Changed lines of the file:
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@@
       (effects (font (size 1.27 1.27)))
     )
-    (property "Value" "MBR0520LT" (at 220.98 80.01 0)
+    (property "Value" "MBR0530-TP" (at 220.98 80.01 0)
       (effects (font (size 1.27 1.27)) hide)
     )
@@
       (effects (font (size 1.27 1.27)))
     )
-    (property "Value" "10R" (at 222.25 27.94 90)
+    (property "Value" "0R" (at 222.25 27.94 90)
       (effects (font (size 1.27 1.27)))
     )
@@
       (effects (font (size 1.27 1.27)))
     )
-    (property "Value" "DMG3415U-7" (at 232.41 24.13 90)
+    (property "Value" "AO3401A" (at 232.41 24.13 90)
       (effects (font (size 1.27 1.27)))
     )
@@
       (effects (font (size 1.27 1.27)) (justify right))
     )
-    (property "Value" "MBR0520LT" (at 214.63 82.2325 90)
+    (property "Value" "MBR0530-TP" (at 214.63 82.2325 90)
       (effects (font (size 1.27 1.27)) (justify right) hide)
     )
@@
       (effects (font (size 1.27 1.27)))
     )
-    (property "Value" "68uH" (at 217.17 63.5 90)
+    (property "Value" "10uH/1A" (at 217.17 63.5 90)
       (effects (font (size 1.27 1.27)))
     )
@@
       (effects (font (size 1.27 1.27)) hide)
     )
+    (property "Mouser" "https://eu.mouser.com/ProductDetail/Murata-Electronics/LQH43PN100M26L?qs=Gufeu08L%2Fl20c%2FBdhusdgA%3D%3D" (at 217.17 60.96 90)
+      (effects (font (size 1.27 1.27)) hide)
+    )
     (pin "1")
     (pin "2")
@@
       (effects (font (size 1.27 1.27)))
     )
-    (property "Value" "MBR0520LT" (at 231.14 80.01 0)
-      (effects (font (size 1.27 1.27)) hide)
-    )
+    (property "Value" "MBR0530-TP" (at 231.14 80.01 0)
+      (effects (font (size 1.27 1.27)) hide)
+    )
